File: Motor.kicad_pcb (KiCad board)
At the start: 2 copper layers, 68.6 x 96.5 mm, 27 parts, among them J1 Battery, J2 TFT Display 128x160, J3 RS232 and Power, J4 IBT_2 H-Bridge, J5 Motor Temperature, J6 Controller Temperature, J7 Rudder Sensor

Commit message: added copyright information
Other:
- board text added: "Author: Timo Birnschein (timo.birnschein@googlemail.com) Copyright by Timo Birnschein 2019"
