File: Motor.sch (KiCad schematic (older format))
At the start: 27 parts, among them J1 Battery, J2 TFT Display 128x160, J3 RS232 and Power, J4 IBT_2 H-Bridge, J5 Motor Temperature, J6 Controller Temperature, J7 Rudder Sensor

Commit message: added copyright information
Parts:
- A1: symbol MCU_Module:Arduino_Nano_v3.x -> Motor-rescue:Arduino_Nano_v3.x-MCU_Module
Other:
- note added: "Author: Timo Birnschein (timo.birnschein@googlemail.com)\nCopyright by Timo Birnschein 2019"
Changed lines of the file:
@@
 EESchema Schematic File Version 4
-LIBS:Motor-cache
-EELAYER 26 0
+EELAYER 30 0
 EELAYER END
 $Descr A4 11693 8268
@@
 $EndDescr
 $Comp
-L MCU_Module:Arduino_Nano_v3.x A1
+L Motor-rescue:Arduino_Nano_v3.x-MCU_Module A1
 U 1 1 5DE324BB
 P 5850 3700
@@
 Text Label 4150 3900 0    50   ~ 0
 A0_DC
+Text Notes 7000 6700 0    50   ~ 0
+Author: Timo Birnschein (timo.birnschein@googlemail.com)\nCopyright by Timo Birnschein 2019
 $EndSCHEMATC
